Commit message: icub_head_epr Gazebo model: remove legs

File: gazebo/models/icub_head_epr/model.urdf (robot description, URDF)
Before this commit: robot icub_head_epr, 102 links, 101 joints
Links:
- removed link l_ankle_1
- removed link l_ankle_2
- removed link l_foot
- removed link l_foot_dh_frame
- removed link l_hip_1
- removed link l_hip_2
- removed link l_hip_3
- removed link l_lower_leg
- removed link l_upper_leg
- removed link l_upper_leg_dh_frame
- removed link r_ankle_1
- removed link r_ankle_2
- removed link r_foot
- removed link r_foot_dh_frame
- removed link r_hip_1
- removed link r_hip_2
- removed link r_hip_3
- removed link r_lower_leg
- removed link r_upper_leg
- removed link r_upper_leg_dh_frame
Joints:
- removed joint l_ankle_pitch
- removed joint l_ankle_roll
- removed joint l_foot_dh_frame_fixed_joint
- removed joint l_foot_ft_sensor
- removed joint l_hip_pitch
- removed joint l_hip_roll
- removed joint l_hip_yaw
- removed joint l_knee
- removed joint l_leg_ft_sensor
- removed joint l_upper_leg_dh_frame_fixed_joint
- removed joint r_ankle_pitch
- removed joint r_ankle_roll
- removed joint r_foot_dh_frame_fixed_joint
- removed joint r_foot_ft_sensor
- removed joint r_hip_pitch
- removed joint r_hip_roll
- removed joint r_hip_yaw
- removed joint r_knee
- removed joint r_leg_ft_sensor
- removed joint r_upper_leg_dh_frame_fixed_joint

Commit message: icub_head_epr Gazebo model: Remove hands and fix torso and arms

File: gazebo/models/icub_head_epr/model.urdf (robot description, URDF)
Before this commit: robot icub_head_epr, 82 links, 81 joints
Links:
- removed link l_hand_index_0
- removed link l_hand_index_1
- removed link l_hand_index_2
- removed link l_hand_index_3
- removed link l_hand_index_tip
- removed link l_hand_little_0
- removed link l_hand_little_1
- removed link l_hand_little_2
- removed link l_hand_little_3
- removed link l_hand_little_tip
- removed link l_hand_middle_0
- removed link l_hand_middle_1
- removed link l_hand_middle_2
- removed link l_hand_middle_3
- removed link l_hand_middle_tip
- removed link l_hand_ring_0
- removed link l_hand_ring_1
- removed link l_hand_ring_2
- removed link l_hand_ring_3
- removed link l_hand_ring_tip
- removed link l_hand_thumb_0
- removed link l_hand_thumb_1
- removed link l_hand_thumb_2
- removed link l_hand_thumb_3
- removed link l_hand_thumb_tip
- removed link r_hand_index_0
- removed link r_hand_index_1
- removed link r_hand_index_2
- removed link r_hand_index_3
- removed link r_hand_index_tip
- removed link r_hand_little_0
- removed link r_hand_little_1
- removed link r_hand_little_2
- removed link r_hand_little_3
- removed link r_hand_little_tip
- removed link r_hand_middle_0
- removed link r_hand_middle_1
- removed link r_hand_middle_2
- removed link r_hand_middle_3
- removed link r_hand_middle_tip
- removed link r_hand_ring_0
- removed link r_hand_ring_1
- removed link r_hand_ring_2
- removed link r_hand_ring_3
- removed link r_hand_ring_tip
- removed link r_hand_thumb_0
- removed link r_hand_thumb_1
- removed link r_hand_thumb_2
- removed link r_hand_thumb_3
- removed link r_hand_thumb_tip
Joints:
- removed joint l_hand_index_0_joint
- removed joint l_hand_index_1_joint
- removed joint l_hand_index_2_joint
- removed joint l_hand_index_3_joint
- removed joint l_hand_index_tip_joint
- removed joint l_hand_little_0_joint
- removed joint l_hand_little_1_joint
- removed joint l_hand_little_2_joint
- removed joint l_hand_little_3_joint
- removed joint l_hand_little_tip_joint
- removed joint l_hand_middle_0_joint
- removed joint l_hand_middle_1_joint
- removed joint l_hand_middle_2_joint
- removed joint l_hand_middle_3_joint
- removed joint l_hand_middle_tip_joint
- removed joint l_hand_ring_0_joint
- removed joint l_hand_ring_1_joint
- removed joint l_hand_ring_2_joint
- removed joint l_hand_ring_3_joint
- removed joint l_hand_ring_tip_joint
- removed joint l_hand_thumb_0_joint
- removed joint l_hand_thumb_1_joint
- removed joint l_hand_thumb_2_joint
- removed joint l_hand_thumb_3_joint
- removed joint l_hand_thumb_tip_joint
- removed joint r_hand_index_0_joint
- removed joint r_hand_index_1_joint
- removed joint r_hand_index_2_joint
- removed joint r_hand_index_3_joint
- removed joint r_hand_index_tip_joint
- removed joint r_hand_little_0_joint
- removed joint r_hand_little_1_joint
- removed joint r_hand_little_2_joint
- removed joint r_hand_little_3_joint
- removed joint r_hand_little_tip_joint
- removed joint r_hand_middle_0_joint
- removed joint r_hand_middle_1_joint
- removed joint r_hand_middle_2_joint
- removed joint r_hand_middle_3_joint
- removed joint r_hand_middle_tip_joint
- removed joint r_hand_ring_0_joint
- removed joint r_hand_ring_1_joint
- removed joint r_hand_ring_2_joint
- removed joint r_hand_ring_3_joint
- removed joint r_hand_ring_tip_joint
- removed joint r_hand_thumb_0_joint
- removed joint r_hand_thumb_1_joint
- removed joint r_hand_thumb_2_joint
- removed joint r_hand_thumb_3_joint
- removed joint r_hand_thumb_tip_joint
- joint l_elbow: type revolute -> fixed
- joint l_shoulder_pitch: type revolute -> fixed
- joint l_shoulder_roll: type revolute -> fixed
- joint l_shoulder_yaw: type revolute -> fixed
- joint l_wrist_pitch: type revolute -> fixed
- joint l_wrist_prosup: type revolute -> fixed
- joint l_wrist_yaw: type revolute -> fixed
- joint r_elbow: type revolute -> fixed
- joint r_shoulder_pitch: type revolute -> fixed
- joint r_shoulder_roll: type revolute -> fixed
- joint r_shoulder_yaw: type revolute -> fixed
- joint r_wrist_pitch: type revolute -> fixed
- joint r_wrist_prosup: type revolute -> fixed
- joint r_wrist_yaw: type revolute -> fixed
- joint torso_pitch: type revolute -> fixed
- joint torso_roll: type revolute -> fixed
- joint torso_yaw: type revolute -> fixed
